File: hw/sch_pcb/USTTHUNDERMILLPCB02A/USTTHUNDERMILLPCB02A.kicad_pcb (KiCad board)
At the start: 2 copper layers, 80 x 80 mm, 0 parts

Commit message: uprava PCB
Routing:
- net GND: vias 0 -> 18
- added copper zone on B.Cu, net GND
- added copper zone on F.Cu, net GND
- removed copper zone on B.Cu, net (none)
- removed copper zone on F.Cu, net (none)
Other:
- outline, holes or cut-outs redrawn

Commit message: uprava PCB
Routing:
- added copper zone on B.Cu, net (none)
- added copper zone on F.Cu, net (none)
- removed copper zone on B.Cu, net GND
- removed copper zone on F.Cu, net GND
Other:
- outline, holes or cut-outs redrawn

Commit message: Edit PCB
Parts:
- added J1: HEADER_1x01, Mlab_Pin_Headers:SMD_1x1, F.Cu at (110.9, 79.7)
Routing:
- added copper zone on B.Cu, net GND
- added copper zone on F.Cu, net GND
- removed copper zone on B.Cu, net (none)
- removed copper zone on F.Cu, net (none)
