File: hw/sch_pcb/USTTHUNDERMILLPCB02A/USTTHUNDERMILLPCB02A.kicad_sch (KiCad schematic)
At the start: 0 parts

Commit message: Edit PCB
Parts:
- added J1: HEADER_1x01, Mlab_Pin_Headers:SMD_1x1, symbol MLAB_HEADER:HEADER_1x01
Connections:
- net GND: now also J1.1
Changed lines of the file:
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@@
-(kicad_sch (version 20210621) (generator eeschema)
+(kicad_sch (version 20210406) (generator eeschema)
   (paper "A4")
+  (wire (pts (xy 62.23 55.245) (xy 62.23 57.15))
+    (stroke (width 0) (type solid) (color 0 0 0 0))
+  )
   (symbol (lib_id "power:GND") (at 62.23 57.15 0) (unit 1)
     (in_bom yes) (on_board yes) (fields_autoplaced)
@@
     (pin "1")
   )
+  (symbol (lib_id "MLAB_HEADER:HEADER_1x01") (at 62.23 50.165 90) (unit 1)
+    (in_bom yes) (on_board yes) (fields_autoplaced)
+    (property "Reference" "J1" (id 0) (at 64.1351 51.3729 90)
+      (effects (font (size 1.524 1.524)) (justify right))
+    )
+    (property "Value" "HEADER_1x01" (id 1) (at 64.1351 54.0805 90)
+      (effects (font (size 1.524 1.524)) (justify right))
+    )
+    (property "Footprint" "Mlab_Pin_Headers:SMD_1x1" (id 2) (at 62.23 50.165 0)
+      (effects (font (size 1.524 1.524)))
+    )
+    (property "Datasheet" "" (id 3) (at 62.23 50.165 0)
+      (effects (font (size 1.524 1.524)))
+    )
+    (pin "1")
+  )
   (sheet_instances
     (path "/" (page "1"))
@@
       (reference "#PWR0101") (unit 1) (value "GND") (footprint "")
     )
+    (path "/ee99d645-9843-4ac9-97bb-387c57c46b94"
+      (reference "J1") (unit 1) (value "HEADER_1x01") (footprint "Mlab_Pin_Headers:SMD_1x1")
+    )
   )
